File: main-board.brd (EAGLE design)
At the start: 134.1 x 43 mm, 0 parts

Commit message: Commit
Parts:
- added ACSW1:C1, ACSW2:C1, ACSW3:C1, ACSW4:C1, ACSW5:C1: (no value), resistor:C050-030X075
- added ACSW1:OK1, ACSW2:OK1, ACSW3:OK1, ACSW4:OK1, ACSW5:OK1: MOC3033M, optocoupler:DIL06
- added ACSW1:R1, ACSW2:R1, ACSW3:R1, ACSW4:R1, ACSW5:R1, R1, R2, R3, R4, R5: 100, resistor:R1206
- added ACSW1:R2, ACSW2:R2, ACSW3:R2, ACSW4:R2, ACSW5:R2: 360, resistor:R1206
- added ACSW1:R3, ACSW2:R3, ACSW3:R3, ACSW4:R3, ACSW5:R3: (no value), resistor:0204/7
- added ACSW1:T1, ACSW2:T1, ACSW3:T1, ACSW4:T1, ACSW5:T1: BT138-V, triac:TO220BV
- added IC2: 74HC595D, 74xx-eu:SO16
Connections:
- new net AC+: ACSW1:OK1.6, ACSW1:R3.2, ACSW1:T1.T2, ACSW2:OK1.6, ACSW2:R3.2, ACSW2:T1.T2, ACSW3:OK1.6, ACSW3:R3.2, ACSW3:T1.T2, ACSW4:OK1.6, ACSW4:R3.2, ACSW4:T1.T2, ACSW5:OK1.6, ACSW5:R3.2, ACSW5:T1.T2
- new net ACSW1:N$1: ACSW1:OK1.1, ACSW1:R1.2
- new net ACSW1:N$2: ACSW1:OK1.4, ACSW1:R2.1, ACSW1:T1.G
- new net ACSW1:N$8: ACSW1:C1.1, ACSW1:R3.1
- new net ACSW2:N$1: ACSW2:OK1.1, ACSW2:R1.2
- new net ACSW2:N$2: ACSW2:OK1.4, ACSW2:R2.1, ACSW2:T1.G
- new net ACSW2:N$8: ACSW2:C1.1, ACSW2:R3.1
- new net ACSW3:N$1: ACSW3:OK1.1, ACSW3:R1.2
- new net ACSW3:N$2: ACSW3:OK1.4, ACSW3:R2.1, ACSW3:T1.G
- new net ACSW3:N$8: ACSW3:C1.1, ACSW3:R3.1
- new net ACSW4:N$1: ACSW4:OK1.1, ACSW4:R1.2
- new net ACSW4:N$2: ACSW4:OK1.4, ACSW4:R2.1, ACSW4:T1.G
- new net ACSW4:N$8: ACSW4:C1.1, ACSW4:R3.1
- new net ACSW5:N$1: ACSW5:OK1.1, ACSW5:R1.2
- new net ACSW5:N$2: ACSW5:OK1.4, ACSW5:R2.1, ACSW5:T1.G
- new net ACSW5:N$8: ACSW5:C1.1, ACSW5:R3.1
- new net GND: ACSW1:OK1.2, ACSW2:OK1.2, ACSW3:OK1.2, ACSW4:OK1.2, ACSW5:OK1.2, IC2.10, IC2.11, IC2.12, IC2.13, IC2.14, IC2.8
- new net N$1: ACSW2:R1.1, R1.2
- new net N$10: IC2.4, R5.1
- new net N$2: IC2.15, R2.1
- new net N$3: IC2.1, R1.1
- new net N$4: ACSW4:R1.1, R4.2
- new net N$5: IC2.2, R3.1
- new net N$6: IC2.3, R4.1
- new net N$7: ACSW1:R1.1, R2.2
- new net N$8: ACSW3:R1.1, R3.2
- new net N$9: ACSW5:R1.1, R5.2
- new net OUT1: ACSW1:C1.2, ACSW1:R2.2, ACSW1:T1.T1
- new net OUT2: ACSW2:C1.2, ACSW2:R2.2, ACSW2:T1.T1
- new net OUT3: ACSW3:C1.2, ACSW3:R2.2, ACSW3:T1.T1
- new net OUT4: ACSW4:C1.2, ACSW4:R2.2, ACSW4:T1.T1
- new net OUT5: ACSW5:C1.2, ACSW5:R2.2, ACSW5:T1.T1
- new net VCC: IC2.16
Other:
- outline, holes or cut-outs redrawn
