File: main-board.brd (EAGLE design)
At the start: 134.1 x 43 mm, 41 parts, among them IC2 74HC595D, SW1:OK1 MOC3033M, SW1:R1 100, SW1:R2 360, SW1:T1 BT138-V

Commit message: update
Parts:
- removed ACSW2:R2, ACSW3:R2, ACSW4:R2, ACSW5:R2, SW1:R2: 360, resistor:R1206
- added ACSW2:R4, ACSW3:R4, ACSW4:R4, ACSW5:R4, SW1:R4: 360, resistor:0204/7
- added C1, C2: (no value), resistor:C4532
- added LAMP1, LAMP2, POWER: (no value), con-molex:KK-156-2
- added MOTOR: (no value), con-molex:KK-156-4
- added SW2, SW3, SW4, SW5, SW6: 1825910-6, Switch:1825910-6
- added U1: LD1117S33TR, IC:SOT-223
- ACSW2:R3, ACSW3:R3, ACSW4:R3, ACSW5:R3, SW1:R3: value (none) -> 39
- R1, R2, R3, R4, R5, R6, R7, R8, R9: value 100 -> 4k7
- moved R5 150.0 mm to (-19.1, -82.5), flipped to the top
- moved R4 144.0 mm to (-19.1, -76.2), flipped to the top
- moved R3 138.2 mm to (-19.1, -69.8), flipped to the top
- moved R2 131.4 mm to (-19.1, -63.5), flipped to the top
- moved R1 129.3 mm to (-19.1, -57.1), flipped to the top
- moved ACSW5:T1 106.9 mm to (52.1, 25.4), turned to 180 degrees
- moved ACSW4:T1 106.3 mm to (63.5, 25.4), turned to 180 degrees
- moved ACSW4:C1 105.4 mm to (64.8, 22.9), turned to 0 degrees
- moved ACSW5:C1 105.0 mm to (53.3, 22.9), turned to 0 degrees
- moved ACSW4:R3 104.2 mm to (63.5, 19.1), turned to 0 degrees
- moved ACSW5:R3 103.9 mm to (52.1, 19.1), turned to 0 degrees
- moved ACSW3:T1 77.1 mm to (39.4, 22.9), turned to 270 degrees
- moved ACSW3:C1 68.7 mm to (33.0, 22.9), turned to 90 degrees
- moved ACSW4:R1 67.6 mm to (105.4, 24.1), flipped to the bottom, turned to 90 degrees
- moved ACSW3:R3 65.1 mm to (30.0, 21.6), turned to 90 degrees
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Connections:
- removed net OUT1: SW1:C1.2, SW1:R2.2, SW1:T1.T1
- removed net OUT2: ACSW2:C1.2, ACSW2:R2.2, ACSW2:T1.T1
- removed net OUT3: ACSW3:C1.2, ACSW3:R2.2, ACSW3:T1.T1
- removed net OUT4: ACSW4:C1.2, ACSW4:R2.2, ACSW4:T1.T1
- removed net OUT5: ACSW5:C1.2, ACSW5:R2.2, ACSW5:T1.T1
- new net +5V: C1.1, U1.3
- new net AC-: LAMP1.2, LAMP2.2, MOTOR.4, POWER.2
- new net LAMP1: ACSW4:C1.2, ACSW4:R4.1, ACSW4:T1.T1, LAMP1.1
- new net LAMP2: ACSW5:C1.2, ACSW5:R4.1, ACSW5:T1.T1, LAMP2.1
- new net M1: MOTOR.1, SW1:C1.2, SW1:R4.1, SW1:T1.T1
- new net M2: ACSW2:C1.2, ACSW2:R4.1, ACSW2:T1.T1, MOTOR.2
- new net M3: ACSW3:C1.2, ACSW3:R4.1, ACSW3:T1.T1, MOTOR.3
- net +3V3: now also C2.1, R5.2, U1.2, U1.4
- net AC+: now also POWER.1
- net ACSW2:N$2: now also ACSW2:R4.2; no longer ACSW2:R2.1
- net ACSW3:N$2: now also ACSW3:R4.2; no longer ACSW3:R2.1
- net ACSW4:N$2: now also ACSW4:R4.2; no longer ACSW4:R2.1
- net ACSW5:N$2: now also ACSW5:R4.2; no longer ACSW5:R2.1
- net GND: now also C1.2, C2.2, SW2.3, SW3.3, SW4.3, SW5.3, SW6.3, U1.1
- net N$1: now also IC2.2; no longer R1.2
- net N$10: now also R1.2, SW2.1; no longer IC2.5
- net N$2: now also R3.1, R4.2, SW5.1; no longer IC2.1, R2.1
- net N$3: now also R4.1, SW6.1; no longer IC2.2, R1.1
- net N$4: now also IC2.4; no longer R4.2
- net N$5: now also R2.1, R3.2, SW4.1; no longer IC2.3, R3.1
- net N$6: now also R1.1, R2.2, SW3.1; no longer IC2.4, R4.1
- net N$7: now also IC2.1; no longer R2.2
- net N$8: now also IC2.3; no longer R3.2
- net N$9: now also IC2.5; no longer R5.2
- net SW1:N$2: now also SW1:R4.2; no longer SW1:R2.1
Routing:
- net AC+: track 0.00 -> 153.2 mm
- net AC-: track 0.00 -> 63.7 mm
- net GND: track 39.2 -> 5.60 mm
- net +3V3: track 31.0 -> 60.4 mm
- net N$13: track 0.00 -> 23.5 mm
- net M3: track 0.00 -> 20.4 mm
- net ACSW4:N$1: track 0.00 -> 17.6 mm
- net LAMP1: track 0.00 -> 17.1 mm
- net N$12: track 0.00 -> 15.7 mm
- net LAMP2: track 0.00 -> 15.3 mm
- net N$4: track 0.00 -> 11.6 mm
- net N$9: track 0.00 -> 8.52 mm
- net N$10: track 8.00 -> 0.00 mm
- net N$6: track 6.73 -> 0.00 mm
- net N$11: track 0.00 -> 6.56 mm
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
Commit message: upd
Parts:
- removed R1, R2, R3, R4, R5: 4k7, resistor:R1206
- removed SW2, SW3, SW4, SW5, SW6: 1825910-6, Switch:1825910-6
- added 5VI, PWRO: (no value), con-molex:KK-156-2
- moved ACSW3:R1 22.2 mm to (95.2, 25.4), turned to 270 degrees
- moved R6 21.7 mm to (116.8, 26.7), turned to 180 degrees
- moved ACSW5:R1 20.5 mm to (95.2, 43.2), turned to 270 degrees
- moved ACSW5:OK1 16.1 mm to (86.4, 43.2)
- moved ACSW2:R1 16.1 mm to (95.2, 16.5), turned to 270 degrees
- moved SW1:OK1 15.7 mm to (86.4, 7.62)
- moved ACSW2:OK1 14.5 mm to (86.4, 16.5)
- moved ACSW4:R1 14.4 mm to (95.2, 34.3), turned to 270 degrees
- moved ACSW3:OK1 13.3 mm to (86.4, 25.4)
- moved ACSW4:OK1 10.6 mm to (86.4, 34.3)
- moved SW1:R1 10.2 mm to (95.2, 7.62), turned to 270 degrees
- moved C2 6.35 mm to (110.5, 41.9)
- moved U1 5.68 mm to (118.1, 41.9), turned to 0 degrees
- moved R9 5.08 mm to (130.8, 27.9), turned to 270 degrees
- moved R7 4.02 mm to (123.2, 26.7)
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Connections:
- removed net N$10: R1.2, R5.1, SW2.1
- removed net N$2: R3.1, R4.2, SW5.1
- removed net N$3: R4.1, SW6.1
- removed net N$5: R2.1, R3.2, SW4.1
- removed net N$6: R1.1, R2.2, SW3.1
- net +3V3: no longer R5.2
- net +5V: now also 5VI.1
- net AC+: now also PWRO.1
- net AC-: now also PWRO.2
- net GND: now also 5VI.2; no longer SW2.3, SW3.3, SW4.3, SW5.3, SW6.3
Routing:
- net GND: track 5.60 -> 87.0 mm
- net N$9: track 8.52 -> 33.4 mm
- net N$8: track 0.00 -> 18.7 mm
- net +3V3: track 60.4 -> 77.6 mm
- net N$4: track 11.6 -> 26.0 mm
- net N$14: track 0.00 -> 12.9 mm
- net ACSW4:N$1: track 17.6 -> 5.54 mm
- net N$1: track 0.00 -> 11.4 mm
- net N$11: track 6.56 -> 17.0 mm
- net +5V: track 4.64 -> 13.6 mm
- net N$7: track 0.00 -> 8.83 mm
- net N$13: track 23.5 -> 15.5 mm
- net SW1:N$1: track 0.00 -> 5.54 mm
- net ACSW2:N$1: track 2.69 -> 5.54 mm
- net N$12: track 15.7 -> 14.4 mm
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- added copper zone on layer 16, net GND
Other:
- board size 134.1 x 43 mm -> 134.1 x 50.9 mm

Commit message: upd
Parts:
- removed ACSW2:C1, ACSW3:C1, ACSW4:C1, ACSW5:C1: (no value), resistor:C050-030X075
- removed ACSW2:R3, ACSW3:R3, ACSW4:R3, ACSW5:R3: 39, resistor:0204/7
- removed ACSW2:R4, ACSW3:R4, ACSW4:R4, ACSW5:R4: 360, resistor:0204/7
- removed ACSW2:T1, ACSW3:T1, ACSW4:T1, ACSW5:T1: BT138-V, triac:TO220BV
- added LED1: (no value), led:SML0603
- added R1: 210, resistor:R0805
- added SW2:C1, SW3:C1, SW4:C1, SW5:C1: (no value), resistor:C050-030X075
- added SW2:R3, SW3:R3, SW4:R3, SW5:R3: 39, resistor:0204/7
- added SW2:R4, SW3:R4, SW4:R4, SW5:R4: 360, resistor:0204/7
- added SW2:T1, SW3:T1, SW4:T1, SW5:T1: BT138-V, triac:TO220BV
- moved PWRO 56.9 mm to (12.7, 43.2)
- moved SW1:R4 34.7 mm to (9.53, 26.0), turned to 0 degrees
- moved SW1:R3 24.5 mm to (9.53, 14.0), turned to 180 degrees
- moved SW1:C1 20.9 mm to (9.53, 17.1), turned to 180 degrees
- moved SW1:T1 13.4 mm to (9.53, 23.5), turned to 0 degrees
- moved LAMP1 4.58 mm to (66.0, 43.2)
- moved LAMP2 4.02 mm to (55.9, 43.2)
- moved MOTOR 3.81 mm to (41.9, 43.2)
- moved POWER 3.81 mm to (24.1, 43.2)
- moved R6 1.27 mm to (115.6, 26.7)
- moved R9 1.27 mm to (129.5, 27.9)
- moved 5VI 1.27 mm to (128.3, 43.2)
- moved C1 1.27 mm to (128.3, 35.6)
- moved C2 1.27 mm to (110.5, 40.6)
- moved R7 1.27 mm to (121.9, 26.7)
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- renumbered ACSW2:OK1 to SW2:OK1, ACSW2:R1 to SW2:R1, ACSW3:OK1 to SW3:OK1, ACSW3:R1 to SW3:R1, ACSW4:OK1 to SW4:OK1, ACSW4:R1 to SW4:R1, ACSW5:OK1 to SW5:OK1, ACSW5:R1 to SW5:R1
Connections:
- net ACSW2:N$1 renamed SW2:N$1
- net ACSW3:N$1 renamed SW3:N$1
- net ACSW4:N$1 renamed SW4:N$1
- net ACSW5:N$1 renamed SW5:N$1
- net SW1:N$2 renamed SW1:ACS
- removed net ACSW2:N$2: ACSW2:R4.2, ACSW2:T1.G, SW2:OK1.4
- removed net ACSW2:N$8: ACSW2:C1.1, ACSW2:R3.1
- removed net ACSW3:N$2: ACSW3:R4.2, ACSW3:T1.G, SW3:OK1.4
- removed net ACSW3:N$8: ACSW3:C1.1, ACSW3:R3.1
- removed net ACSW4:N$2: ACSW4:R4.2, ACSW4:T1.G, SW4:OK1.4
- removed net ACSW4:N$8: ACSW4:C1.1, ACSW4:R3.1
- removed net ACSW5:N$2: ACSW5:R4.2, ACSW5:T1.G, SW5:OK1.4
- removed net ACSW5:N$8: ACSW5:C1.1, ACSW5:R3.1
- new net N$2: LED1.A, R1.2
- new net SW2:ACS: SW2:OK1.4, SW2:R4.2, SW2:T1.G
- new net SW2:N$8: SW2:C1.1, SW2:R3.1
- new net SW3:ACS: SW3:OK1.4, SW3:R4.2, SW3:T1.G
- new net SW3:N$8: SW3:C1.1, SW3:R3.1
- new net SW4:ACS: SW4:OK1.4, SW4:R4.2, SW4:T1.G
- new net SW4:N$8: SW4:C1.1, SW4:R3.1
- new net SW5:ACS: SW5:OK1.4, SW5:R4.2, SW5:T1.G
- new net SW5:N$8: SW5:C1.1, SW5:R3.1
- net +3V3: now also R1.1
- net AC+: now also SW2:R3.2, SW2:T1.T2, SW3:R3.2, SW3:T1.T2, SW4:R3.2, SW4:T1.T2, SW5:R3.2, SW5:T1.T2; no longer ACSW2:R3.2, ACSW2:T1.T2, ACSW3:R3.2, ACSW3:T1.T2, ACSW4:R3.2, ACSW4:T1.T2, ACSW5:R3.2, ACSW5:T1.T2
- net GND: now also LED1.C
- net LAMP1: now also SW5:C1.2, SW5:R4.1, SW5:T1.T1; no longer ACSW4:C1.2, ACSW4:R4.1, ACSW4:T1.T1
- net LAMP2: now also SW4:C1.2, SW4:R4.1, SW4:T1.T1; no longer ACSW5:C1.2, ACSW5:R4.1, ACSW5:T1.T1
- net M2: now also SW2:C1.2, SW2:R4.1, SW2:T1.T1; no longer ACSW2:C1.2, ACSW2:R4.1, ACSW2:T1.T1
- net M3: now also SW3:C1.2, SW3:R4.1, SW3:T1.T1; no longer ACSW3:C1.2, ACSW3:R4.1, ACSW3:T1.T1
Routing:
- net AC+: track 153.2 -> 306.5 mm
- net SW1:ACS: track 0.00 -> 84.6 mm
- net SW2:ACS: track 0.00 -> 75.7 mm
- net SW3:ACS: track 0.00 -> 67.7 mm
- net M1: track 3.81 -> 50.0 mm
- net M2: track 0.00 -> 40.9 mm
- net SW4:ACS: track 0.00 -> 35.7 mm
- net SW5:ACS: track 0.00 -> 30.9 mm
- net LAMP2: track 15.3 -> 40.9 mm
- net AC-: track 63.7 -> 75.7 mm
- net M3: track 20.4 -> 31.3 mm
- net ACSW3:N$2: track 4.86 -> 0.00 mm
- net ACSW5:N$8: track 4.86 -> 0.00 mm
- net ACSW4:N$8: track 4.86 -> 0.00 mm
- net SW5:N$8: track 0.00 -> 4.34 mm
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
Commit message: upd
Parts:
- added SV1: (no value), con-lstb:MA03-1
- moved IC2 3.81 mm to (106.4, 19.1)
Connections:
- net +3V3: now also SV1.2
- net BTX: now also SV1.3
- net GND: now also SV1.1
Routing:
- net GND: track 87.5 -> 177.5 mm
- net +3V3: track 76.3 -> 85.1 mm
- net BTX: track 0.00 -> 6.30 mm
- net N$9: track 33.4 -> 30.0 mm
- net N$4: track 26.0 -> 23.1 mm
- net N$8: track 18.7 -> 16.2 mm
- net N$7: track 8.83 -> 11.2 mm
- net CLT: track 5.61 -> 7.69 mm
- net N$1: track 11.4 -> 9.33 mm
- net CSCK: track 5.92 -> 7.55 mm
- net CDT: track 5.84 -> 6.72 mm
