File: main-board.sch (EAGLE design)
At the start: 6 parts, among them IC1 74LS595D

Commit message: Commit
Parts:
- removed IC1: 74LS595D, 74xx-us:74LS595D
- removed LAMP1, LAMP2, PWR, PWR2: 5566-2, omez-packs:5566-2
- removed MOTOR: 5566-4, omez-packs:5566-4
- added IC2: 74HC595D, 74xx-eu:74HC595D
- added R1, R2, R3, R4, R5: 100, resistor:R-EU_R1206
Connections:
- removed net LAMP1: LAMP1-2.S
- removed net LAMP2: LAMP2-2.S
- removed net MS1: MOTOR-2.S
- removed net MS2: MOTOR-3.S
- removed net MS3: MOTOR-4.S
- removed net PWR+: PWR-2.S, PWR2-2.S
- removed net PWR-: LAMP1-1.S, LAMP2-1.S, MOTOR-1.S, PWR-1.S, PWR2-1.S
- new net AC+: R3.2
- new net AC-: R2.2
- new net CTL: R1.1
- new net GND: IC2A.G, IC2A.RCK, IC2A.SCK, IC2A.SCL, IC2A.SER
- new net N$10: IC2A.QE, R5.1
- new net N$6: IC2A.QD, R4.1
- new net N$7: R2.2
- new net N$8: R3.1, R3.2
- new net N$9: R5.2
- net N$1: now also R1.2; no longer IC1A.QA
- net N$2: now also IC2A.QA, R2.1; no longer IC1A.QB
- net N$3: now also IC2A.QB, R1.1; no longer IC1A.QC
- net N$4: now also R4.2; no longer IC1A.QD
- net N$5: now also IC2A.QC, R3.1; no longer IC1A.QE
