File: main-board.sch (EAGLE design)
At the start: 11 parts, among them IC2 74HC595D

Commit message: update
Parts:
- added C1, C2: (no value), resistor:C-USC4532
- added LAMP1, LAMP2, POWER: (no value), con-molex:KK-156-2
- added MOTOR: (no value), con-molex:KK-156-4
- added SW2, SW3, SW4, SW5, SW6: 1825910-6, Switch:1825910-6
- added U1: LD1117S33TR, IC:LD1117S33TR
- R1, R2, R3, R4, R5, R6, R7, R8, R9: value 100 -> 4k7
Connections:
- new net +5V: C1.1, U1.IN
- new net LAMP1: LAMP1-1.S
- new net LAMP2: LAMP2-1.S
- new net M1: MOTOR-1.S
- new net M2: MOTOR-2.S
- new net M3: MOTOR-3.S
- net +3V3: now also C2.1, R5.2, U1.4, U1.OUT
- net AC+: now also POWER-1.S
- net AC-: now also C1.2, LAMP1-2.S, LAMP2-2.S, MOTOR-4.S, POWER-2.S, R4.1; no longer R2.2
- net GND: now also C1.2, C2.2, SW2.3, SW3.3, SW4.3, SW5.3, SW6.3, U1.ADJ/GND
- net N$1: now also IC2A.QC
- net N$10: now also R1.2, SW2.1; no longer IC2A.QF
- net N$2: now also R3.1, R4.2, SW5.1; no longer IC2A.QB, R2.1
- net N$3: now also R4.1, SW6.1; no longer IC2A.QC, R1.1
- net N$4: now also IC2A.QE; no longer R4.2
- net N$5: now also R2.1, R3.2, SW4.1; no longer IC2A.QD, R3.1
- net N$6: now also R1.1, R2.2, SW3.1; no longer IC2A.QE, R4.1
- net N$7: now also IC2A.QB; no longer R2.2
- net N$8: now also C1.1, IC2A.QD; no longer R3.2
- net N$9: now also IC2A.QF; no longer R5.2

Commit message: upd
Parts:
- removed R1, R2, R3, R4, R5: 4k7, resistor:R-EU_R1206
- removed SW2, SW3, SW4, SW5, SW6: 1825910-6, Switch:1825910-6
- added 5VI, PWRO: (no value), con-molex:KK-156-2
Connections:
- removed net CTL: R1.1
- removed net N$10: R1.2, R5.1, SW2.1
- removed net N$2: R3.1, R4.2, SW5.1
- removed net N$3: R4.1, SW6.1
- removed net N$5: R2.1, R3.2, SW4.1
- removed net N$6: R1.1, R2.2, SW3.1
- net +3V3: no longer R5.2
- net +5V: now also 5VI-1.S
- net AC+: now also PWRO-1.S; no longer R3.2
- net AC-: now also PWRO-2.S; no longer R4.1
- net GND: now also 5VI-2.S; no longer SW2.3, SW3.3, SW4.3, SW5.3, SW6.3
- net N$1: no longer R1.2
- net N$8: no longer R3.1

Commit message: upd
Parts:
- added LED1: (no value), led:LEDSML0603
- added R1: 210, resistor:R-EU_R0805
Connections:
- new net CTL: R1.1
- new net N$2: LED1.A, R1.2
- net +3V3: now also R1.1
- net GND: now also LED1.C
- net N$1: now also R1.2

Commit message: upd
Parts:
- added SV1: (no value), con-lstb:MA03-1
Connections:
- net +3V3: now also SV1.2
- net BTX: now also SV1.3
- net GND: now also SV1.1
Changed lines of the file:
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@@
 <drawing>
 <settings>
-<setting alwaysvectorfont="no"/>
+<setting alwaysvectorfont="yes"/>
 <setting verticaltext="up"/>
 </settings>
@@
 <part name="+3V6" library="supply1" library_urn="urn:adsk.eagle:library:371" deviceset="+3V3" device=""/>
 <part name="GND6" library="supply1" library_urn="urn:adsk.eagle:library:371" deviceset="GND" device=""/>
+<part name="SV1" library="con-lstb" library_urn="urn:adsk.eagle:library:162" deviceset="MA03-1" device="" package3d_urn="urn:adsk.eagle:package:8339/1"/>
+<part name="GND7" library="supply1" library_urn="urn:adsk.eagle:library:371" deviceset="GND" device=""/>
+<part name="+3V7" library="supply1" library_urn="urn:adsk.eagle:library:371" deviceset="+3V3" device=""/>
 </parts>
 <sheets>
@@
 <attribute name="VALUE" x="-73.66" y="40.64" size="1.778" layer="96"/>
 </instance>
+<instance part="SV1" gate="G$1" x="5.08" y="15.24" smashed="yes">
+<attribute name="VALUE" x="3.81" y="7.62" size="1.778" layer="96"/>
+<attribute name="NAME" x="3.81" y="21.082" size="1.778" layer="95"/>
+</instance>
+<instance part="GND7" gate="1" x="15.24" y="7.62" smashed="yes">
+<attribute name="VALUE" x="12.7" y="5.08" size="1.778" layer="96"/>
+</instance>
+<instance part="+3V7" gate="G$1" x="15.24" y="25.4" smashed="yes">
+<attribute name="VALUE" x="12.7" y="20.32" size="1.778" layer="96" rot="R90"/>
+</instance>
 </instances>
 <busses>
@@
 <wire x1="-71.12" y1="45.72" x2="-71.12" y2="48.26" width="0.1524" layer="91"/>
 </segment>
+<segment>
+<pinref part="SV1" gate="G$1" pin="1"/>
+<pinref part="GND7" gate="1" pin="GND"/>
+<wire x1="12.7" y1="12.7" x2="15.24" y2="12.7" width="0.1524" layer="91"/>
+<wire x1="15.24" y1="12.7" x2="15.24" y2="10.16" width="0.1524" layer="91"/>
+</segment>
 </net>
 <net name="AC+" class="1">
@@
 <label x="-48.26" y="60.96" size="1.778" layer="95"/>
 </segment>
+<segment>
+<pinref part="SV1" gate="G$1" pin="3"/>
+<wire x1="12.7" y1="17.78" x2="20.32" y2="17.78" width="0.1524" layer="91"/>
+<wire x1="22.86" y1="17.78" x2="20.32" y2="17.78" width="0.1524" layer="91"/>
+<label x="22.86" y="17.78" size="1.778" layer="95" rot="R180"/>
+</segment>
 </net>
 <net name="N$11" class="0">
@@
 <wire x1="-71.12" y1="68.58" x2="-71.12" y2="71.12" width="0.1524" layer="91"/>
 </segment>
-</net>
+<segment>
+<pinref part="SV1" gate="G$1" pin="2"/>
+<pinref part="+3V7" gate="G$1" pin="+3V3"/>
+<wire x1="12.7" y1="15.24" x2="15.24" y2="15.24" width="0.1524" layer="91"/>
+<wire x1="15.24" y1="15.24" x2="15.24" y2="22.86" width="0.1524" layer="91"/>
+</segment>
+</net>
