File: keyboard.brd (EAGLE design)
At the start: 94 x 21.3 mm, 10 parts

Commit message: upd
Parts:
- moved R1 32.3 mm to (17.3, -19.8)
- moved R2 32.3 mm to (30.0, -19.8)
- moved R3 32.3 mm to (42.7, -19.8)
- moved R4 32.3 mm to (55.4, -19.8)
- moved R5 32.3 mm to (4.57, -19.8)
- moved BT_L 11.9 mm to (81.7, 9.40)
- moved BT_OFF 7.41 mm to (11.7, 9.40)
- moved BT_S3 7.08 mm to (64.2, 9.40)
- moved BT_S1 2.68 mm to (29.2, 9.40)
- moved BT_S2 2.36 mm to (46.7, 9.40)
Connections:
- net N$10 renamed BTX

Commit message: upd
Parts:
- removed BT_L, BT_OFF: 1825910-6, Switch:1825910-6
- added BT_LIGHT, BT_S0: 1825910-6, Switch:1825910-6
- added SV1: (no value), con-lstb:MA03-1
- moved R1 48.7 mm to (-26.0, 2.54), turned to 0 degrees
- moved R2 44.5 mm to (-8.50, 2.54), turned to 0 degrees
- moved R3 39.5 mm to (8.50, 0.00), turned to 0 degrees
- moved R4 36.9 mm to (26.0, 2.54), turned to 0 degrees
- moved BT_S1 30.7 mm to (0.00, 0.00)
- moved BT_S2 30.7 mm to (17.5, 0.00)
- moved BT_S3 30.7 mm to (35.0, 0.00)
- moved R5 23.7 mm to (8.50, 3.56), turned to 180 degrees
Connections:
- net +3V3: now also SV1.2
- net BTX: now also BT_LIGHT.1, BT_LIGHT.2, SV1.3; no longer BT_OFF.1
- net GND: now also BT_LIGHT.3, BT_LIGHT.4, BT_S0.3, BT_S0.4, BT_S1.4, BT_S2.4, BT_S3.4, SV1.1; no longer BT_L.3, BT_OFF.3
- net N$2: now also BT_S2.1, BT_S2.2; no longer BT_S3.1
- net N$3: now also BT_S3.1, BT_S3.2; no longer BT_L.1
- net N$5: now also BT_S1.1, BT_S1.2; no longer BT_S2.1
- net N$6: now also BT_S0.1, BT_S0.2; no longer BT_S1.1
Routing:
- net GND: track 0.00 -> 115.4 mm, vias 0 -> 1
- net BTX: track 0.00 -> 50.7 mm
- net N$2: track 0.00 -> 16.3 mm
- net N$5: track 0.00 -> 15.8 mm
- net N$6: track 0.00 -> 15.2 mm
- net N$3: track 0.00 -> 10.1 mm
- net +3V3: track 0.00 -> 4.00 mm
Other:
- board size 94 x 21.3 mm -> 102 x 16.2 mm

Commit message: upd
Parts:
- removed BT_LIGHT, BT_S0, BT_S1, BT_S2, BT_S3: 1825910-6, Switch:1825910-6
- added S1, S2, S3, S4, S5: MOMENTARY-SWITCH-SPST-PTH-6.0MM, SparkFun-Switches:TACTILE_SWITCH_PTH_6.0MM
- moved R1 2.54 mm to (-26.0, 0.00)
- moved R2 2.54 mm to (-8.50, 0.00)
- moved R4 2.54 mm to (26.0, 0.00)
Connections:
- net BTX: now also S1.1; no longer BT_LIGHT.1, BT_LIGHT.2
- net GND: now also S1.3, S2.3, S3.3, S4.3, S5.3; no longer BT_LIGHT.3, BT_LIGHT.4, BT_S0.3, BT_S0.4, BT_S1.3, BT_S1.4, BT_S2.3, BT_S2.4, BT_S3.3, BT_S3.4
- net N$2: now also S4.1; no longer BT_S2.1, BT_S2.2
- net N$3: now also S5.1; no longer BT_S3.1, BT_S3.2
- net N$5: now also S3.1; no longer BT_S1.1, BT_S1.2
- net N$6: now also S2.1; no longer BT_S0.1, BT_S0.2
Routing:
- net GND: track 115.4 -> 128.5 mm, vias 1 -> 0
- net BTX: track 50.7 -> 63.4 mm
- net N$3: track 10.1 -> 5.26 mm
- net N$6: track 15.2 -> 16.5 mm
- added copper zone on layer 16, net GND
