File: keyboard.sch (EAGLE design)
At the start: 10 parts

Commit message: upd
Connections:
- net N$10 renamed BTX
Changed lines of the file:
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@@
 <setting verticaltext="up"/>
 </settings>
-<grid distance="0.1" unitdist="inch" unit="inch" style="lines" multiple="1" display="yes" altdistance="0.01" altunitdist="inch" altunit="inch"/>
+<grid distance="0.1" unitdist="inch" unit="inch" style="lines" multiple="1" display="no" altdistance="0.01" altunitdist="inch" altunit="inch"/>
 <layers>
 <layer number="1" name="Top" color="4" fill="1" visible="no" active="no"/>
@@
 </segment>
 </net>
-<net name="N$10" class="0">
+<net name="BTX" class="0">
 <segment>
 <pinref part="R1" gate="G$1" pin="2"/>
@@
 <wire x1="5.08" y1="73.66" x2="0" y2="73.66" width="0.1524" layer="91"/>
 <junction x="0" y="73.66"/>
-</segment>
-</net>
+<wire x1="0" y1="73.66" x2="-12.7" y2="73.66" width="0.1524" layer="91"/>
+<label x="-12.7" y="73.66" size="1.778" layer="95"/>
+</segment>
+</net>

Commit message: upd
Parts:
- removed BT_L: 1825910-6, Switch:1825910-6
- added BT_S0: 1825910-6, Switch:1825910-6
- added SV1: (no value), con-lstb:MA03-1
- renumbered BT_OFF to BT_LIGHT
Connections:
- net +3V3: now also SV1.2
- net BTX: now also BT_LIGHT.2, SV1.3
- net GND: now also BT_LIGHT.4, BT_S0.3, BT_S0.4, BT_S1.4, BT_S2.4, BT_S3.4, SV1.1; no longer BT_L.3
- net N$2: now also BT_S2.1, BT_S2.2; no longer BT_S3.1
- net N$3: now also BT_S3.1, BT_S3.2; no longer BT_L.1
- net N$5: now also BT_S1.1, BT_S1.2; no longer BT_S2.1
- net N$6: now also BT_S0.1, BT_S0.2; no longer BT_S1.1
Other:
- moved on the sheet: BT_S1, BT_S2, BT_S3

Commit message: upd
Parts:
- removed BT_LIGHT, BT_S0, BT_S1, BT_S2, BT_S3: 1825910-6, Switch:1825910-6
- added S1, S2, S3, S4, S5: MOMENTARY-SWITCH-SPST-PTH-6.0MM, SparkFun-Switches:MOMENTARY-SWITCH-SPST-PTH-6.0MM
Connections:
- net BTX: now also S1.1; no longer BT_LIGHT.1, BT_LIGHT.2
- net GND: now also S1.2, S2.2, S3.2, S4.2, S5.2; no longer BT_LIGHT.3, BT_LIGHT.4, BT_S0.3, BT_S0.4, BT_S1.3, BT_S1.4, BT_S2.3, BT_S2.4, BT_S3.3, BT_S3.4
- net N$2: now also S4.1; no longer BT_S2.1, BT_S2.2
- net N$3: now also S5.1; no longer BT_S3.1, BT_S3.2
- net N$5: now also S3.1; no longer BT_S1.1, BT_S1.2
- net N$6: now also S2.1; no longer BT_S0.1, BT_S0.2
